Commit message: sensors FINISHED

File: body.urdf (robot description, URDF)
Before this commit: robot robot, 3 links, 2 joints
Links:
- removed link Link0
- removed link Link1
- removed link Link2
- added link BackLeg, mass 1; collision box size=1 1 1; visual box size=1 1 1
- added link FrontLeg, mass 1; collision box size=1 1 1; visual box size=1 1 1
- added link Torso, mass 1; collision box size=1 1 1; visual box size=1 1 1
Joints:
- removed joint Link0_Link1
- removed joint Link1_Link2
- added joint Torso_BackLeg: type revolute, parent Torso, child BackLeg, origin xyz=1 0 1.0 rpy=0 0 0, axis 0 1 0, limit lower=-3.14159 upper=3.14159 effort=0.0 velocity=0.0
- added joint Torso_FrontLeg: type revolute, parent Torso, child FrontLeg, origin xyz=2 0 1 rpy=0 0 0, axis 0 1 0, limit lower=-3.14159 upper=3.14159 effort=0.0 velocity=0.0

Commit message: Quadruped not working

File: body.urdf (robot description, URDF)
Before this commit: robot robot, 3 links, 2 joints
Links:
- added link LeftLeg, mass 1; collision box size=1 0.2 0.2; visual box size=1 0.2 0.2
- link BackLeg: geometry collision box size=0.2 1 0.2; visual box size=0.2 1 0.2
- link FrontLeg: geometry collision box size=0.2 1 0.2; visual box size=0.2 1 0.2
Joints:
- added joint Torso_LeftLeg: type revolute, parent Torso, child LeftLeg, origin xyz=-0.5 0 1 rpy=0 0 0, axis 0 1 0, limit lower=-3.14159 upper=3.14159 effort=0.0 velocity=0.0
- joint Torso_BackLeg: axis 0 1 0 -> 1 0 0; origin xyz=1 0 1.0 rpy=0 0 0 -> xyz=0 -0.5 1.0 rpy=0 0 0
- joint Torso_FrontLeg: axis 0 1 0 -> 1 0 0; origin xyz=2 0 1 rpy=0 0 0 -> xyz=0 0.5 1 rpy=0 0 0

Commit message: Part N COMPLETE quadruped working

File: body.urdf (robot description, URDF)
Before this commit: robot robot, 4 links, 3 joints
Links:
- added link BackLowerLeg, mass 1; collision box size=0.2 0.2 1; visual box size=0.2 0.2 1
- added link FrontLowerLeg, mass 1; collision box size=0.2 0.2 1; visual box size=0.2 0.2 1
- added link LeftLowerLeg, mass 1; collision box size=0.2 0.2 1; visual box size=0.2 0.2 1
- added link RightLeg, mass 1; collision box size=1 0.2 0.2; visual box size=1 0.2 0.2
- added link RightLowerLeg, mass 1; collision box size=0.2 0.2 1; visual box size=0.2 0.2 1
Joints:
- added joint BackLeg_BackLowerLeg: type revolute, parent BackLeg, child BackLowerLeg, origin xyz=0 -1 0 rpy=0 0 0, axis 1 0 0, limit lower=-3.14159 upper=3.14159 effort=0.0 velocity=0.0
- added joint FrontLeg_FrontLowerLeg: type revolute, parent FrontLeg, child FrontLowerLeg, origin xyz=0 1 0 rpy=0 0 0, axis 1 0 0, limit lower=-3.14159 upper=3.14159 effort=0.0 velocity=0.0
- added joint LeftLeg_LeftLowerLeg: type revolute, parent LeftLeg, child LeftLowerLeg, origin xyz=-1 0 0 rpy=0 0 0, axis 0 1 0, limit lower=-3.14159 upper=3.14159 effort=0.0 velocity=0.0
- added joint RightLeg_RightLowerLeg: type revolute, parent RightLeg, child RightLowerLeg, origin xyz=1 0 0 rpy=0 0 0, axis 0 1 0, limit lower=-3.14159 upper=3.14159 effort=0.0 velocity=0.0
- added joint Torso_RightLeg: type revolute, parent Torso, child RightLeg, origin xyz=0.5 0 1 rpy=0 0 0, axis 0 1 0, limit lower=-3.14159 upper=3.14159 effort=0.0 velocity=0.0

Commit message: updates 1

File: body.urdf (robot description, URDF)
Before this commit: robot robot, 9 links, 8 joints
Links:
- added link LefterLeg, mass 1; collision box size=1 0.2 0.2; visual box size=1 0.2 0.2
- added link LefterLowerLeg, mass 1; collision box size=0.2 0.2 1; visual box size=0.2 0.2 1
- added link RighterLeg, mass 1; collision box size=1 0.2 0.2; visual box size=1 0.2 0.2
- added link RighterLowerLeg, mass 1; collision box size=0.2 0.2 1; visual box size=0.2 0.2 1
- link Torso: geometry collision box size=0.7 2 1; visual box size=0.7 2 1
Joints:
- added joint LefterLeg_LefterLowerLeg: type revolute, parent LefterLeg, child LefterLowerLeg, origin xyz=-1 0.3 0 rpy=0 0 0, axis 0 1 0, limit lower=-3.14159 upper=3.14159 effort=0.0 velocity=0.0
- added joint RighterLeg_RighterLowerLeg: type revolute, parent RighterLeg, child RighterLowerLeg, origin xyz=1 0.3 0 rpy=0 0 0, axis 0 1 0, limit lower=-3.14159 upper=3.14159 effort=0.0 velocity=0.0
- added joint Torso_LefterLeg: type revolute, parent Torso, child LefterLeg, origin xyz=-0.5 0.3 2 rpy=0 0 0, axis 0 1 0, limit lower=-3.14159 upper=3.14159 effort=0.0 velocity=0.0
- added joint Torso_RighterLeg: type revolute, parent Torso, child RighterLeg, origin xyz=0.5 0.3 2 rpy=0 0 0, axis 0 1 0, limit lower=-3.14159 upper=3.14159 effort=0.0 velocity=0.0
- joint LeftLeg_LeftLowerLeg: origin xyz=-1 0 0 rpy=0 0 0 -> xyz=-1 -0.9 0 rpy=0 0 0
- joint RightLeg_RightLowerLeg: origin xyz=1 0 0 rpy=0 0 0 -> xyz=1 -0.9 0 rpy=0 0 0
- joint Torso_BackLeg: origin xyz=0 -0.5 1.0 rpy=0 0 0 -> xyz=0 -0.5 2.0 rpy=0 0 0
- joint Torso_FrontLeg: origin xyz=0 0.5 1 rpy=0 0 0 -> xyz=0 0.5 2 rpy=0 0 0
- joint Torso_LeftLeg: origin xyz=-0.5 0 1 rpy=0 0 0 -> xyz=-0.5 0.35 2 rpy=0 0 0
- joint Torso_RightLeg: origin xyz=0.5 0 1 rpy=0 0 0 -> xyz=0.5 0.35 2 rpy=0 0 0

Commit message: updates 3

File: body.urdf (robot description, URDF)
Before this commit: robot robot, 13 links, 12 joints
Links:
- removed link BackLowerLeg
- removed link FrontLowerLeg
- removed link LeftLeg
- removed link LeftLowerLeg
- removed link LefterLeg
- removed link LefterLowerLeg
- removed link RightLeg
- removed link RightLowerLeg
- removed link RighterLeg
- removed link RighterLowerLeg
- link BackLeg: geometry collision box size=1 1 1; visual box size=1 1 1
- link FrontLeg: geometry collision box size=1 1 1; visual box size=1 1 1
- link Torso: geometry collision box size=1 1 1; visual box size=1 1 1
Joints:
- removed joint BackLeg_BackLowerLeg
- removed joint FrontLeg_FrontLowerLeg
- removed joint LeftLeg_LeftLowerLeg
- removed joint LefterLeg_LefterLowerLeg
- removed joint RightLeg_RightLowerLeg
- removed joint RighterLeg_RighterLowerLeg
- removed joint Torso_LeftLeg
- removed joint Torso_LefterLeg
- removed joint Torso_RightLeg
- removed joint Torso_RighterLeg
- joint Torso_BackLeg: axis 1 0 0 -> 0 1 0; origin xyz=0 -0.5 2.0 rpy=0 0 0 -> xyz=1 0 1.0 rpy=0 0 0
- joint Torso_FrontLeg: axis 1 0 0 -> 0 1 0; origin xyz=0 0.5 2 rpy=0 0 0 -> xyz=2 0 1 rpy=0 0 0

Commit message: car 1

File: body.urdf (robot description, URDF)
Before this commit: robot robot, 3 links, 2 joints
Links:
- removed link BackLeg
- removed link FrontLeg
- added link LeftLeg, mass 2; collision box size=0.5 0.5 0.5; visual box size=0.5 0.5 0.5
- added link LefterLeg, mass 2; collision box size=0.5 0.5 0.5; visual box size=0.5 0.5 0.5
- added link RightLeg, mass 2; collision box size=0.5 0.5 0.5; visual box size=0.5 0.5 0.5
- added link RighterLeg, mass 2; collision box size=0.5 0.5 0.5; visual box size=0.5 0.5 0.5
- link Torso: mass 1 -> 2; geometry collision box size=0.7 2 1; visual box size=0.7 2 1
Joints:
- removed joint Torso_BackLeg
- removed joint Torso_FrontLeg
- added joint Torso_LeftLeg: type revolute, parent Torso, child LeftLeg, origin xyz=-0.5 0.35 1.5 rpy=0 0 0, axis 1 0 0, limit lower=-3.14159 upper=3.14159 effort=0.0 velocity=0.0
- added joint Torso_LefterLeg: type revolute, parent Torso, child LefterLeg, origin xyz=-0.5 0.3 1.5 rpy=0 0 0, axis 1 0 0, limit lower=-3.14159 upper=3.14159 effort=0.0 velocity=0.0
- added joint Torso_RightLeg: type revolute, parent Torso, child RightLeg, origin xyz=0.5 0.35 1.5 rpy=0 0 0, axis 0 1 0, limit lower=-3.14159 upper=3.14159 effort=0.0 velocity=0.0
- added joint Torso_RighterLeg: type revolute, parent Torso, child RighterLeg, origin xyz=0.5 0.3 1.5 rpy=0 0 0, axis 0 1 0, limit lower=-3.14159 upper=3.14159 effort=0.0 velocity=0.0

Commit message: 8 wheeler

File: body.urdf (robot description, URDF)
Before this commit: robot robot, 5 links, 4 joints
Links:
- removed link LeftLeg
- removed link LefterLeg
- removed link RightLeg
- removed link RighterLeg
- added link LeftBackOne, mass 2; collision box size=0.5 0.5 0.5; visual box size=0.5 0.5 0.5
- added link LeftBackTwo, mass 2; collision box size=0.5 0.5 0.5; visual box size=0.5 0.5 0.5
- added link LeftFrontOne, mass 2; collision box size=0.5 0.5 0.5; visual box size=0.5 0.5 0.5
- added link LeftFrontTwo, mass 2; collision box size=0.5 0.5 0.5; visual box size=0.5 0.5 0.5
- added link RightBackOne, mass 2; collision box size=0.5 0.5 0.5; visual box size=0.5 0.5 0.5
- added link RightBackTwo, mass 2; collision box size=0.5 0.5 0.5; visual box size=0.5 0.5 0.5
- added link RightFrontOne, mass 2; collision box size=0.5 0.5 0.5; visual box size=0.5 0.5 0.5
- added link RightFrontTwo, mass 2; collision box size=0.5 0.5 0.5; visual box size=0.5 0.5 0.5
Joints:
- removed joint Torso_LeftLeg
- removed joint Torso_LefterLeg
- removed joint Torso_RightLeg
- removed joint Torso_RighterLeg
- added joint Torso_LeftBackOne: type revolute, parent Torso, child LeftBackOne, origin xyz=-0.5 -0.75 1.5 rpy=0 0 0, axis 1 0 0, limit lower=-3.14159 upper=3.14159 effort=0.0 velocity=0.0
- added joint Torso_LeftBackTwo: type revolute, parent Torso, child LeftBackTwo, origin xyz=-0.5 -0.7 1.5 rpy=0 0 0, axis 1 0 0, limit lower=-3.14159 upper=3.14159 effort=0.0 velocity=0.0
- added joint Torso_LeftFrontOne: type revolute, parent Torso, child LeftFrontOne, origin xyz=-0.5 0.75 1.5 rpy=0 0 0, axis 1 0 0, limit lower=-3.14159 upper=3.14159 effort=0.0 velocity=0.0
- added joint Torso_LeftFrontTwo: type revolute, parent Torso, child LeftFrontTwo, origin xyz=-0.5 0.7 1.5 rpy=0 0 0, axis 1 0 0, limit lower=-3.14159 upper=3.14159 effort=0.0 velocity=0.0
- added joint Torso_RightBackOne: type revolute, parent Torso, child RightBackOne, origin xyz=0.5 -0.75 1.5 rpy=0 0 0, axis 1 0 0, limit lower=-3.14159 upper=3.14159 effort=0.0 velocity=0.0
- added joint Torso_RightBackTwo: type revolute, parent Torso, child RightBackTwo, origin xyz=0.5 -0.75 1.5 rpy=0 0 0, axis 1 0 0, limit lower=-3.14159 upper=3.14159 effort=0.0 velocity=0.0
- added joint Torso_RightFrontOne: type revolute, parent Torso, child RightFrontOne, origin xyz=0.5 0.75 1.5 rpy=0 0 0, axis 1 0 0, limit lower=-3.14159 upper=3.14159 effort=0.0 velocity=0.0
- added joint Torso_RightFrontTwo: type revolute, parent Torso, child RightFrontTwo, origin xyz=0.5 0.7 1.5 rpy=0 0 0, axis 1 0 0, limit lower=-3.14159 upper=3.14159 effort=0.0 velocity=0.0

Commit message: Last commit before adding new pyrosim

File: body.urdf (robot description, URDF)
Before this commit: robot robot, 9 links, 8 joints
Links:
- removed link LeftBackTwo
- removed link LeftFrontTwo
- removed link RightBackTwo
- removed link RightFrontTwo
Joints:
- removed joint Torso_LeftBackTwo
- removed joint Torso_LeftFrontTwo
- removed joint Torso_RightBackTwo
- removed joint Torso_RightFrontTwo

Commit message: Car driving and working

File: body.urdf (robot description, URDF)
Before this commit: robot robot, 5 links, 4 joints
Links:
- added link Sphere1, mass .05; collision sphere radius=.4; visual mesh filename=textured_sphere_smooth.obj scale=.4 .4 .4
- added link Sphere2, mass .05; collision sphere radius=.4; visual mesh filename=textured_sphere_smooth.obj scale=.4 .4 .4
Joints:
- added joint Torso_Sphere1: type revolute, parent Torso, child Sphere1, origin xyz=-0.5 0.75 1.5 rpy=0 0 0, axis 1 0 0, limit lower=-3.14159 upper=3.14159 effort=0.0 velocity=0.0
- added joint Torso_Sphere2: type revolute, parent Torso, child Sphere2, origin xyz=0.5 0.75 1.5 rpy=0 0 0, axis 1 0 0, limit lower=-3.14159 upper=3.14159 effort=0.0 velocity=0.0

Commit message: SNAKE DONE 1

File: body.urdf (robot description, URDF)
Before this commit: robot robot, 7 links, 6 joints
Links:
- removed link LeftBackOne
- removed link LeftFrontOne
- removed link RightBackOne
- removed link RightFrontOne
- removed link Sphere1
- removed link Sphere2
- removed link Torso
- added link Link0, mass 2; collision box size=0.6744050801615727 0.5235529253041188 1.0440909874152702; visual box size=0.6744050801615727 0.5235529253041188 1.0440909874152702
- added link Link1, mass 2; collision box size=1.1463601376711954 0.8149627382057472 0.8620922040700858; visual box size=1.1463601376711954 0.8149627382057472 0.8620922040700858
- added link Link2, mass 2; collision box size=0.8756742652598635 0.8385630050783598 0.9167630536205469; visual box size=0.8756742652598635 0.8385630050783598 0.9167630536205469
- added link Link3, mass 2; collision box size=1.0078067320623765 1.1566305979245188 1.1585364314099689; visual box size=1.0078067320623765 1.1566305979245188 1.1585364314099689
- added link Link4, mass 2; collision box size=1.062862474396045 0.8260732929430717 0.8729153047318574; visual box size=1.062862474396045 0.8260732929430717 0.8729153047318574
- added link Link5, mass 2; collision box size=0.8812760143213579 1.1762219913005327 1.050159279515259; visual box size=0.8812760143213579 1.1762219913005327 1.050159279515259
Joints:
- removed joint Torso_LeftBackOne
- removed joint Torso_LeftFrontOne
- removed joint Torso_RightBackOne
- removed joint Torso_RightFrontOne
- removed joint Torso_Sphere1
- removed joint Torso_Sphere2
- added joint Link0_Link1: type revolute, parent Link0, child Link1, origin xyz=0 0 1.25 rpy=0 0 0, axis 0 0 1, limit lower=-3.14159 upper=3.14159 effort=0.0 velocity=0.0
- added joint Link1_Link2: type revolute, parent Link1, child Link2, origin xyz=1.1463601376711954 0 0 rpy=0 0 0, axis 1 0 0, limit lower=-3.14159 upper=3.14159 effort=0.0 velocity=0.0
- added joint Link2_Link3: type revolute, parent Link2, child Link3, origin xyz=0.8756742652598635 0 0 rpy=0 0 0, axis 0 0 1, limit lower=-3.14159 upper=3.14159 effort=0.0 velocity=0.0
- added joint Link3_Link4: type revolute, parent Link3, child Link4, origin xyz=1.0078067320623765 0 0 rpy=0 0 0, axis 0 1 0, limit lower=-3.14159 upper=3.14159 effort=0.0 velocity=0.0
- added joint Link4_Link5: type revolute, parent Link4, child Link5, origin xyz=1.062862474396045 0 0 rpy=0 0 0, axis 0 0 1, limit lower=-3.14159 upper=3.14159 effort=0.0 velocity=0.0

Commit message: Final Snake

File: body.urdf (robot description, URDF)
Before this commit: robot robot, 6 links, 5 joints
Links:
- added link Link6, mass 2; collision box size=1.2013621571726956 1.1985298791925445 0.9982336509263713; visual box size=1.2013621571726956 1.1985298791925445 0.9982336509263713
- link Link0: geometry collision box size=1.3383338887042413 1.404229668973226 0.940566976735709; visual box size=1.3383338887042413 1.404229668973226 0.940566976735709
- link Link1: geometry collision box size=1.197905764429005 1.0751268012377049 0.8437229782051123; visual box size=1.197905764429005 1.0751268012377049 0.8437229782051123
- link Link2: geometry collision box size=1.1600193490874628 0.799068595954973 1.0388013223685388; visual box size=1.1600193490874628 0.799068595954973 1.0388013223685388
- link Link3: geometry collision box size=0.990380434834317 1.1519735367959831 0.9259619831813178; visual box size=0.990380434834317 1.1519735367959831 0.9259619831813178
- link Link4: geometry collision box size=1.1690849399556489 1.1926335438564193 1.2428453792504999; visual box size=1.1690849399556489 1.1926335438564193 1.2428453792504999
- link Link5: geometry collision box size=1.1257898781768363 0.7854632505414276 0.9418907471598751; visual box size=1.1257898781768363 0.7854632505414276 0.9418907471598751
Joints:
- added joint Link5_Link6: type revolute, parent Link5, child Link6, origin xyz=1.1257898781768363 0 0 rpy=0 0 0, axis 0 1 0, limit lower=-3.14159 upper=3.14159 effort=0.0 velocity=0.0
- joint Link0_Link1: axis 0 0 1 -> 1 0 0
- joint Link1_Link2: axis 1 0 0 -> 0 0 1; origin xyz=1.1463601376711954 0 0 rpy=0 0 0 -> xyz=1.197905764429005 0 0 rpy=0 0 0
- joint Link2_Link3: origin xyz=0.8756742652598635 0 0 rpy=0 0 0 -> xyz=1.1600193490874628 0 0 rpy=0 0 0
- joint Link3_Link4: axis 0 1 0 -> 0 0 1; origin xyz=1.0078067320623765 0 0 rpy=0 0 0 -> xyz=0.990380434834317 0 0 rpy=0 0 0
- joint Link4_Link5: axis 0 0 1 -> 0 1 0; origin xyz=1.062862474396045 0 0 rpy=0 0 0 -> xyz=1.1690849399556489 0 0 rpy=0 0 0

Commit message: ASSIGNMENT7DONE

File: body.urdf (robot description, URDF)
Before this commit: robot robot, 7 links, 6 joints
Links:
- link Link0: geometry collision box size=1.5491021543156787 1.7690745225327509 1.842085996557957; visual box size=1.5491021543156787 1.7690745225327509 1.842085996557957
- link Link1: geometry collision box size=1.122264425970961 1.0957876906363202 0.851290370676565; visual box size=1.122264425970961 1.0957876906363202 0.851290370676565
- link Link2: geometry collision box size=0.8745652813096928 0.7525925552917452 1.190297827919471; visual box size=0.8745652813096928 0.7525925552917452 1.190297827919471
- link Link3: geometry collision box size=0.8433291050822883 0.9720587303271553 0.8932832278498106; visual box size=0.8433291050822883 0.9720587303271553 0.8932832278498106
- link Link4: geometry collision box size=0.9715464736137374 0.8730197739176984 0.8273933969874687; visual box size=0.9715464736137374 0.8730197739176984 0.8273933969874687
- link Link5: geometry collision box size=0.9501995650029554 1.0803331497202096 0.8010768929438093; visual box size=0.9501995650029554 1.0803331497202096 0.8010768929438093
- link Link6: geometry collision box size=1.0057761118766086 1.2110437634535014 1.129988906743648; visual box size=1.0057761118766086 1.2110437634535014 1.129988906743648
Joints:
- removed joint Link2_Link3
- removed joint Link3_Link4
- removed joint Link5_Link6
- added joint Link1_Link3: type revolute, parent Link1, child Link3, origin xyz=0.851290370676565 0 0.8433291050822883 rpy=0 0 0, axis 0 1 0, limit lower=-3.14159 upper=3.14159 effort=0.0 velocity=0.0
- added joint Link2_Link4: type revolute, parent Link2, child Link4, origin xyz=0.851290370676565 0.8730197739176984 0.7525925552917452 rpy=0 0 0, axis 1 0 0, limit lower=-3.14159 upper=3.14159 effort=0.0 velocity=0.0
- added joint Link4_Link6: type revolute, parent Link4, child Link6, origin xyz=0.851290370676565 1.2110437634535014 0.7525925552917452 rpy=0 0 0, axis 0 0 1, limit lower=-3.14159 upper=3.14159 effort=0.0 velocity=0.0
- joint Link0_Link1: axis 1 0 0 -> 0 0 1; origin xyz=0 0 1.25 rpy=0 0 0 -> xyz=0.851290370676565 0 0 rpy=0 0 0
- joint Link1_Link2: origin xyz=1.197905764429005 0 0 rpy=0 0 0 -> xyz=0.851290370676565 0 0.7525925552917452 rpy=0 0 0
- joint Link4_Link5: axis 0 1 0 -> 0 0 1; origin xyz=1.1690849399556489 0 0 rpy=0 0 0 -> xyz=0.851290370676565 0.9501995650029554 0.7525925552917452 rpy=0 0 0
