Commit message: Created body file but haven't linked

File: body1.urdf (robot description, URDF)
Before this commit: robot robot, 4 links, 3 joints
Links:
- link Link0: geometry collision box size=0.9864392280079097 0.9128783521234223 1.0753537983144508; visual box size=0.9864392280079097 0.9128783521234223 1.0753537983144508
- link Link1: geometry collision box size=1.187669501901936 0.9977137631980306 1.097856539313064; visual box size=1.187669501901936 0.9977137631980306 1.097856539313064
- link Link2: geometry collision box size=1.245686708275349 1.2056838834209824 1.0039803824888496; visual box size=1.245686708275349 1.2056838834209824 1.0039803824888496
- link Link3: geometry collision box size=1.0938473526656993 0.9684850951640248 0.8495955005515744; visual box size=1.0938473526656993 0.9684850951640248 0.8495955005515744
Joints:
- removed joint Link1_Link3
- added joint Link0_Link3: type revolute, parent Link0, child Link3, origin xyz=0.9128783521234223 0 0 rpy=0 0 0, axis 0 1 0, limit lower=-3.14159 upper=3.14159 effort=0.0 velocity=0.0
- joint Link0_Link1: axis 0 1 0 -> 1 0 0; origin xyz=0.9783928453019648 0 0 rpy=0 0 0 -> xyz=1.0753537983144508 0 0 rpy=0 0 0
- joint Link1_Link2: axis 1 0 0 -> 0 1 0; origin xyz=0 0 1.1945248763076342 rpy=0 0 0 -> xyz=0 0 0.9977137631980306 rpy=0 0 0
